File: circuit/remote-programmer/remote-programmer.kicad_sch (KiCad schematic)
At the start: 22 parts, among them J1 Raspberry Pi W, J10 SPI-5V, J11 SPI-3.3V, J12 I2C-5V, J2 USB_C, J3 PICO0, J4 I2C-5V, J5 AVR, J6 I2C-5V, J7 I2C-5V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

Commit message: .
Parts:
- added J13: FTDI, symbol Connector_Generic:Conn_01x06
- added LS1: Beeper, symbol Device:Speaker
- added R3: 220, symbol Device:R
Connections:
- net GND: now also J1.36 (Pin_36), U2.7 (A5), LS1.2
- net RGND: now also J13.6 (Pin_6), R3.1; no longer DS2.2 (LEDA)
- net RX-5V: now also J13.3 (Pin_3)
- net TX-5V: now also J13.2 (Pin_2)
- net at U2.14 (B5): now also LS1.1
- new net: DS2.2 (LEDA), R3.2
- no-connect marks 4 -> 7
Other:
- moved on the sheet: RV1

Commit message: .
Parts:
- removed Q1: 2N2222, Package_TO_SOT_THT:TO-92_Inline, symbol Transistor_BJT:2N3904
- removed U1, U2: FXMA108, Package_DFN_QFN:WQFN-20-1EP_2.5x4.5mm_P0.5mm_EP1x2.9mm, symbol Logic_LevelTranslator:FXMA108
- added U1, U2, U3, U4: LEVEL SHIFT, Package_SO:SOIC-14_3.9x8.7mm_P1.27mm, symbol Logic_LevelTranslator:TXB0104D
Connections:
- net +3.3V: now also U1.14 (VCCB), U2.14 (VCCB), U3.14 (VCCB), U4.14 (VCCB)
- net +5V: now also U1.1 (VCCA), U2.1 (VCCA), U3.1 (VCCA), U4.1 (VCCA); no longer J1.2 (Pin_2), J2.1 (VBUS), SW1.3
- net AVR-MISO-5V: now also U2.3 (A2)
- net AVR-MOSI-5V: now also U2.2 (A1)
- net CLK-5V: now also U2.4 (A3)
- net CS0-5V: now also U1.5 (A4)
- net CS1-5V: now also U4.4 (A3)
- net GND: now also U1.7 (GND), U2.7 (GND), U3.7 (GND), U4.7 (GND); no longer J1.36 (Pin_36)
- net GPIO10 (MOSI): now also U1.13 (B1)
- net GPIO11 (SCK): now also U1.11 (B3)
- net GPIO12 (RST): now also U2.10 (B4)
- net GPIO14 (TX): now also U3.13 (B1)
- net GPIO15 (RX): now also U3.12 (B2)
- net GPIO18 (AVMOSI): now also U2.13 (B1)
- net GPIO2 (SDA): now also U4.12 (B2)
- net GPIO23 (AVMISO): now also U2.12 (B2)
- net GPIO24 (SWCLK): now also U2.11 (B3)
- net GPIO3 (SCL): now also U4.13 (B1)
- net GPIO7 (CE1): now also U4.11 (B3)
- net GPIO8 (CE0): now also U1.10 (B4)
- net GPIO9 (MISO): now also U1.12 (B2)
- net MISO-5V: now also U1.3 (A2)
- net MOSI-5V: now also U1.2 (A1)
- net RST-5V: now also U2.5 (A4)
- net RX-5V: now also U3.3 (A2)
- net SCK-5V: now also U1.4 (A3)
- net SCL-5V: now also U4.2 (A1)
- net SDA-5V: now also U4.3 (A2)
- net TX-5V: now also U3.2 (A1)
- net at LS1.1: now also U3.4 (A3)
- new net GPIO16 (BEEP): J1.36 (Pin_36), U3.11 (B3)
- new net R5V: J1.2 (Pin_2), J2.1 (VBUS), SW1.3
- no-connect marks 7 -> 15
Other:
- moved on the sheet: D1, J13, LS1, Q2, R1

Commit message: .
Parts:
- removed Q2: 2N2222, Package_TO_SOT_THT:TO-92_Inline, symbol Transistor_BJT:2N3904
- added Q1: 2N2222, Package_TO_SOT_THT:TO-92_Inline, symbol Transistor_BJT:2N3904
- added R4: 10K, symbol Device:R
- R2: value 4.7k -> 4.7K
Connections:
- net +3.3V: now also Q1.1 (E), R4.1; no longer J1.1 (Pin_1), U1.14 (VCCB), U2.14 (VCCB), U3.14 (VCCB), U4.14 (VCCB)
- net +5V: now also R2.1, U3.5 (A4); no longer U1.1 (VCCA), U2.1 (VCCA), U3.1 (VCCA), U4.1 (VCCA)
- net GND: now also R4.2
- net GPIO01 (PWR): now also U3.10 (B4); no longer R2.1
- net R5V: now also U1.1 (VCCA), U2.1 (VCCA), U3.1 (VCCA), U4.1 (VCCA)
- net at R2.2: now also Q1.2 (B)
- new net R3.3V: J1.1 (Pin_1), Q1.3 (C), U1.14 (VCCB), U2.14 (VCCB), U3.14 (VCCB), U4.14 (VCCB)
- no-connect marks 15 -> 13
Other:
- moved on the sheet: D1, R1

Commit message: .
Parts:
- added R5: 10k, symbol Device:R
- added SW2: RESET, symbol Switch:SW_Push
Connections:
- net GND: now also SW2.1
- net GPIO12 (RST): now also R5.2, SW2.2
- net R3.3V: now also U3.10 (B4), R5.1
- net GPIO01 (PWR): no longer names the net of J1.28 (Pin_28)
- net GPIO01 (PWR): no longer U3.10 (B4)
Other:
- moved on the sheet: D1, LS1, R1

Commit message: .
Connections:
- net GPIO11 (SCK): now also J1.23 (Pin_23); no longer J1.15 (Pin_15)
- net GPIO9 (MISO): now also J1.21 (Pin_21); no longer J1.17 (Pin_17)
Changed lines of the file:
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@@
+	(wire
+		(pts
+			(xy 17.78 46.99) (xy 35.56 46.99)
+		)
+		(stroke
+			(width 0)
+			(type default)
+		)
+	)
 	(wire
 		(pts
@@
 	(wire
 		(pts
-			(xy 17.78 57.15) (xy 35.56 57.15)
-		)
-		(stroke
-			(width 0)
-			(type default)
-		)
-	)
-	(wire
-		(pts
 			(xy 140.97 88.9) (xy 123.19 88.9)
 		)
@@
 	(wire
 		(pts
+			(xy 17.78 49.53) (xy 35.56 49.53)
+		)
+		(stroke
+			(width 0)
+			(type default)
+		)
+	)
+	(wire
+		(pts
 			(xy 107.95 140.97) (xy 107.95 144.78)
 		)
@@
 		(pts
 			(xy 139.7 152.4) (xy 139.7 153.67)
-		)
-		(stroke
-			(width 0)
-			(type default)
-		)
-	)
-	(wire
-		(pts
-			(xy 17.78 54.61) (xy 35.56 54.61)
 		)
 		(stroke
@@
 		)
 	)
+	(label "GPIO11 (SCK)"
+		(at 33.02 46.99 180)
+		(effects
+			(font
+				(size 1.27 1.27)
+			)
+			(justify right bottom)
+		)
+	)
 	(label "CS0"
 		(at 254 60.96 180)
@@
 		)
 	)
-	(label "GPIO9 (MISO)"
-		(at 33.02 54.61 180)
-		(effects
-			(font
-				(size 1.27 1.27)
-			)
-			(justify right bottom)
-		)
-	)
 	(label "GPIO15 (RX)"
 		(at 179.07 33.02 180)
@@
 		)
 	)
+	(label "GPIO9 (MISO)"
+		(at 33.02 49.53 180)
+		(effects
+			(font
+				(size 1.27 1.27)
+			)
+			(justify right bottom)
+		)
+	)
 	(label "R5V"
 		(at 49.53 74.93 0)
@@
 		)
 	)
-	(label "GPIO11 (SCK)"
-		(at 33.02 57.15 180)
-		(effects
-			(font
-				(size 1.27 1.27)
-			)
-			(justify right bottom)
-		)
-	)

Commit message: .
Connections:
- net GPIO0 (D4): no longer J1.27 (Pin_27)
- net GPIO19 (D4): now reaches J1.35 (Pin_35)
Changed lines of the file:
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@@
+	(wire
+		(pts
+			(xy 17.78 31.75) (xy 35.56 31.75)
+		)
+		(stroke
+			(width 0)
+			(type default)
+		)
+	)
 	(wire
 		(pts
@@
 		(pts
 			(xy 140.97 83.82) (xy 123.19 83.82)
-		)
-		(stroke
-			(width 0)
-			(type default)
-		)
-	)
-	(wire
-		(pts
-			(xy 17.78 41.91) (xy 35.56 41.91)
 		)
 		(stroke
@@
 		)
 	)
+	(label "GPIO19 (D4)"
+		(at 33.02 31.75 180)
+		(effects
+			(font
+				(size 1.27 1.27)
+			)
+			(justify right bottom)
+		)
+	)
 	(label "GPIO23 (AVMISO)"
 		(at 49.53 57.15 0)
@@
 		(effects
 			(font
-				(size 1.27 1.27)
-			)
-			(justify right bottom)
-		)
-	)
-	(label "GPIO0 (D4)"
-		(at 33.02 41.91 180)
-		(effects
-			(font

Commit message: .
Parts:
- removed J10: SPI-5V, symbol Connector_Generic:Conn_01x06
- removed J11: SPI-3.3V, symbol Connector_Generic:Conn_01x06
- removed J8: PWR_5V, symbol Connector_Generic:Conn_01x02
- removed J9: PWR_3.3V, symbol Connector_Generic:Conn_01x02
- added J10: SPI-5V, symbol Connector_Generic:Conn_01x05
- added J11: SPI-3.3V, symbol Connector_Generic:Conn_01x05
- added J14: PWR-5V, symbol Connector_Generic:Conn_01x03
- added J15: PWR-3.3V, symbol Connector_Generic:Conn_01x03
- J12: value I2C-5V -> UART-3.3V
- J3: value PICO0 -> SWD
- J6: value I2C-5V -> I2C-3.3V
- J7: value I2C-5V -> UART-5V
- R5: value 10k -> 10K
Connections:
- net +3.3V: now also J15.1 (Pin_1)
- net +5V: now also J14.1 (Pin_1)
- net CS0: now also J11.4 (Pin_4)
- net CS0-5V: now also J10.4 (Pin_4)
- net GND: now also J10.5 (Pin_5), J11.5 (Pin_5), J14.3 (Pin_3), J15.3 (Pin_3)
- net GPIO12 (RST): now also J15.2 (Pin_2)
- net MISO: now also J11.2 (Pin_2)
- net MISO-5V: now also J10.2 (Pin_2)
- net MOSI: now also J11.1 (Pin_1)
- net MOSI-5V: now also J10.1 (Pin_1)
- net RST-5V: now also J14.2 (Pin_2)
- net SCK: now also J11.3 (Pin_3)
- net SCK-5V: now also J10.3 (Pin_3)

Commit message: .
Parts:
- removed D1: LED, symbol Device:LED
- removed DS2: HY1602E, Display:HY1602E, symbol Display_Character:HY1602E
- removed J1: Raspberry Pi W, symbol Connector_Generic:Conn_02x20_Odd_Even
- removed J10: SPI-5V, symbol Connector_Generic:Conn_01x05
- removed J11: SPI-3.3V, symbol Connector_Generic:Conn_01x05
- removed J12: UART-3.3V, symbol Connector_Generic:Conn_01x03
- removed J13: FTDI, symbol Connector_Generic:Conn_01x06
- removed J14: PWR-5V, symbol Connector_Generic:Conn_01x03
- removed J15: PWR-3.3V, symbol Connector_Generic:Conn_01x03
- removed J2: USB_C, symbol Connector:USB_A
- removed J4: I2C-5V, symbol Connector_Generic:Conn_01x03
- removed J6: I2C-3.3V, symbol Connector_Generic:Conn_01x03
- removed J7: UART-5V, symbol Connector_Generic:Conn_01x03
- removed LS1: Beeper, symbol Device:Speaker
- removed Q1: 2N2222, Package_TO_SOT_THT:TO-92_Inline, symbol Transistor_BJT:2N3904
- removed R1, R3: 220, symbol Device:R
- removed R2: 4.7K, symbol Device:R
- removed R4, R5: 10K, symbol Device:R
- removed RV1: Pot, symbol Device:R_Potentiometer
- removed SW1: SW_DPST, symbol Switch:SW_DPST
- removed SW2: RESET, symbol Switch:SW_Push
- removed U1, U2, U3, U4: LEVEL SHIFT, Package_SO:SOIC-14_3.9x8.7mm_P1.27mm, symbol Logic_LevelTranslator:TXB0104D
- added D3, D4, D5, D6: 1N4148, Diode_THT:D_DO-35_SOD27_P7.62mm_Horizontal, symbol Diode:1N4148
- added D7: LED, symbol Device:LED
- added J8: Raspberry Pi W, symbol Connector_Generic:Conn_02x20_Odd_Even
- added J9: USB_C, symbol Connector:USB_A
- added LS2: Beeper, symbol Device:Speaker
- added Q2: 2N2222, Package_TO_SOT_THT:TO-92_Inline, symbol Transistor_BJT:2N3904
- added R10: 220, symbol Device:R
- added R6, R8: 10K, symbol Device:R
- added R7: 4.7K, symbol Device:R
- added SW3: SW_DPST, symbol Switch:SW_DPST
- added SW4: RESET, symbol Switch:SW_Push
- added U5: 0.91 OLED, Package_TO_SOT_SMD:SOT-23-5, symbol Memory_EEPROM:24AA02E-OT
Connections:
- net AVR-MISO-5V is gone; now on net MISO: J5.5 (Pin_5)
- net TX-5V is gone; now on net +3.3V: J5.9 (Pin_9)
- net +3.3V: now also Q2.1 (E), R8.1
- net +5V: now also D7.2 (A), R7.1, SW3.4
- net GND: now also LS2.2, R10.2, R8.2, SW3.2, SW4.1, U5.2 (V_{SS}); no longer J5.7 (Pin_7), J5.8 (Pin_8)
- net GPIO10 (MOSI): now also D4.2 (A), J8.19 (Pin_19)
- net GPIO12 (RST): now also J8.32 (Pin_32), R6.2, SW4.2
- net GPIO14 (TX): now also J8.8 (Pin_8)
- net GPIO15 (RX): now also J8.10 (Pin_10)
- net GPIO16 (BEEP): now also J8.36 (Pin_36), LS2.1
- net GPIO2 (SDA): now also D6.2 (A), J8.3 (Pin_3), U5.3 (SDA)
- net GPIO24 (SWCLK): now also J8.18 (Pin_18)
- net GPIO25 (SWIO): now also J8.22 (Pin_22)
- net GPIO3 (SCL): now also D5.2 (A), J8.5 (Pin_5), U5.1 (SCL)
- net GPIO8 (CE0): now also J8.24 (Pin_24)
- net GPIO9 (MISO): now also D3.2 (A), J8.21 (Pin_21)
- net MISO: now also D3.1 (K)
- net R3.3V: now also J8.1 (Pin_1), Q2.3 (C), R6.1, U5.4 (V_{CC})
- net R5V: now also J8.2 (Pin_2), J9.1 (VBUS), SW3.3
- net RGND: now also J8.6 (Pin_6), J9.4 (GND), SW3.1
- net RX: now also J5.7 (Pin_7)
- net TX: now also J5.8 (Pin_8)
- net AVR-MOSI-5V renamed MOSI/SDA
- net MOSI/SDA: now also D4.1 (K), D6.1 (K)
- net CLK-5V renamed CLK/SCL
- net CLK/SCL: now also D5.1 (K), J8.23 (Pin_23)
- net RST-5V renamed RST
- net RX-5V renamed CS
- new net: Q2.2 (B), R7.2
- new net: D7.1 (K), R10.1
- no-connect marks 13 -> 0
Other:
- moved on the sheet: J3, J5
