File: circuit/remote-programmer/remote-programmer.kicad_sch (KiCad schematic)
At the start: 18 parts, among them J3 SWD, J5 AVR, J8 Raspberry Pi W, J9 USB_C, Q2 2N2222, SW3 SW_DPST, SW4 RESET, U5 0.91 OLED

Commit message: .
Parts:
- removed D3, D4, D5, D6: 1N4148, Diode_THT:D_DO-35_SOD27_P7.62mm_Horizontal, symbol Diode:1N4148
Connections:
- net CLK/SCL: no longer J8.23 (Pin_23)
- new net GPIO11 (SCK): J8.23 (Pin_23)

Commit message: .
Parts:
- added J1: Conn_01x04, symbol Connector_Generic:Conn_01x04
- added SERIAL: RESET, symbol Switch:SW_Push
- added U1: FDTI module, Package_SO:SOIC-8_3.9x4.9mm_P1.27mm, symbol Interface_USB:CH330N
Connections:
- net +3.3V: now also J1.3 (Pin_3), U1.5 (VCC)
- net GND: now also J1.4 (Pin_4), SERIAL.2, U1.3 (GND)
- net RX: now also U1.7 (RXD)
- net TX: now also U1.6 (TXD)
- net GPIO23 (SERIAL): now reaches J8.16 (Pin_16)
- net GPIO23 (SERIAL): now also SERIAL.1
- net CLK/SCL renamed CLK
- net MOSI/SDA renamed MOSI
- new net SCL: J1.1 (Pin_1)
- new net SDA: J1.2 (Pin_2)
- no-connect marks 0 -> 4
Other:
- moved on the sheet: D7, J3, J5, J8, J9, LS2, Q2, R10, R6, R7, R8, SW3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

Commit message: .
Parts:
- removed U1: FDTI module, Package_SO:SOIC-8_3.9x4.9mm_P1.27mm, symbol Interface_USB:CH330N
- added J13: FTDI, symbol Connector_Generic:Conn_01x06
Connections:
- net GND: no longer J1.4 (Pin_4), J3.2 (Pin_2), J5.6 (Pin_6)
- net RGND: now also J1.4 (Pin_4), J3.2 (Pin_2), J5.6 (Pin_6), J13.6 (Pin_6)
- net RX: now also J13.3 (Pin_3)
- net TX: now also J13.2 (Pin_2)
- net GPIO8 (CE0) renamed GPIO8 (CS)
- no-connect marks 4 -> 3
Other:
- added sheet Converter (converter.kicad_sch)
