File: circuit/remote-programmer/remote-programmer.kicad_sch (KiCad schematic)
At the start: 17 parts, among them J1 Conn_01x04, J13 FTDI, J3 SWD, J5 AVR, J8 Raspberry Pi W, J9 USB_C, Q2 2N2222, SW3 SW_DPST, SW4 RESET, U5 0.91 OLED

Commit message: .
Connections:
- net GPIO07 (SERIAL): now reaches J8.26 (Pin_26)
- net GPIO07 (SERIAL): now also SERIAL.1
- net GPIO23 (SERIAL): no longer names the net of J8.16 (Pin_16)
- net GPIO23 (SERIAL): no longer SERIAL.1
Changed lines of the file:
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@@
-	(wire
-		(pts
-			(xy 104.14 88.9) (xy 123.19 88.9)
-		)
-		(stroke
-			(width 0)
-			(type default)
-		)
-	)
 	(wire
 		(pts
@@
 	(wire
 		(pts
+			(xy 123.19 88.9) (xy 123.19 76.2)
+		)
+		(stroke
+			(width 0)
+			(type default)
+		)
+	)
+	(wire
+		(pts
 			(xy 205.74 50.8) (xy 205.74 59.69)
 		)
@@
 		(pts
 			(xy 147.32 153.67) (xy 147.32 154.94)
+		)
+		(stroke
+			(width 0)
+			(type default)
+		)
+	)
+	(wire
+		(pts
+			(xy 123.19 76.2) (xy 104.14 76.2)
 		)
 		(stroke
@@
 		)
 	)
-	(label "GPIO23 (SERIAL)"
-		(at 105.41 88.9 0)
+	(label "GPIO07 (SERIAL)"
+		(at 105.41 76.2 0)
 		(effects
 			(font
